File: pcb_designs/PCB Draft 1/4-7-2024.kicad_pcb (KiCad board)
At the start: 2 copper layers, 69.7 x 97 mm, 19 parts, among them J1 Joystick_F_TH, J2 Joystick_B_TH, J3 Conn_01x17_Pin, J4 Conn_01x17_Pin, SW1 Left_Trigger, SW10 D_Pad_DOWN, SW11 D_Pad_LEFT, SW12 D_Pad_RIGHT, SW13 A_Button, SW14 X_Button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

Commit message: :construction: rewire ground connection
Routing:
- net /GND: track 356.7 -> 369.7 mm
Changed lines of the file:
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@@
+	)
+	(segment
+		(start 167.64 116.84)
+		(end 167.64 121.52)
+		(width 0.2)
+		(layer "F.Cu")
+		(net 4)
 	)
 	(segment
@@
 	)
 	(segment
+		(start 161.795 78.74)
+		(end 161.795 77.673683)
+		(width 0.2)
+		(layer "F.Cu")
+		(net 4)
+	)
+	(segment
+		(start 177.76 116.84)
+		(end 182.88 116.84)
+		(width 0.2)
+		(layer "F.Cu")
+		(net 4)
+	)
+	(segment
+		(start 182.88 111.76)
+		(end 175.26 104.14)
+		(width 0.2)
+		(layer "F.Cu")
+		(net 4)
+	)
+	(segment
+		(start 147.32 71.12)
+		(end 147.32 66.04)
+		(width 0.2)
+		(layer "F.Cu")
+		(net 4)
+	)
+	(segment
+		(start 172.72 139.7)
+		(end 172.72 137.16)
+		(width 0.2)
+		(layer "F.Cu")
+		(net 4)
+	)
+	(segment
+		(start 160.02 93.98)
+		(end 160.02 99.06)
+		(width 0.2)
+		(layer "F.Cu")
+		(net 4)
+	)
+	(segment
+		(start 137.16 71.12)
+		(end 147.32 71.12)
+		(width 0.2)
+		(layer "F.Cu")
+		(net 4)
+	)
+	(segment
+		(start 180.34 78.74)
+		(end 182.88 78.74)
+		(width 0.2)
+		(layer "F.Cu")
+		(net 4)
+	)
+	(segment
+		(start 175.26 93.98)
+		(end 175.26 99.06)
+		(width 0.2)
+		(layer "F.Cu")
+		(net 4)
+	)
+	(segment
+		(start 177.8 78.74)
+		(end 180.34 78.74)
+		(width 0.2)
+		(layer "F.Cu")
+		(net 4)
+	)
+	(segment
+		(start 182.88 121.92)
+		(end 182.88 116.84)
+		(width 0.2)
+		(layer "F.Cu")
+		(net 4)
+	)
+	(segment
+		(start 182.88 116.84)
+		(end 182.88 111.76)
+		(width 0.2)
+		(layer "F.Cu")
+		(net 4)
+	)
+	(segment
+		(start 137.16 124.46)
+		(end 167.64 124.46)
+		(width 0.2)
+		(layer "F.Cu")
+		(net 4)
+	)
+	(segment
+		(start 142.2 66.04)
+		(end 147.32 66.04)
+		(width 0.2)
+		(layer "F.Cu")
+		(net 4)
+	)
+	(segment
+		(start 152.4 55.88)
+		(end 152.4 66.04)
+		(width 0.2)
+		(layer "F.Cu")
+		(net 4)
+	)
+	(segment
+		(start 175.26 93.98)
+		(end 160.02 93.98)
+		(width 0.2)
+		(layer "F.Cu")
+		(net 4)
+	)
+	(segment
+		(start 167.64 124.46)
+		(end 167.64 139.7)
+		(width 0.2)
+		(layer "F.Cu")
+		(net 4)
+	)
+	(segment
+		(start 157.48 134.62)
+		(end 157.48 139.7)
+		(width 0.2)
+		(layer "F.Cu")
+		(net 4)
+	)
+	(segment
+		(start 182.88 66.04)
+		(end 180.3 66.04)
+		(width 0.2)
+		(layer "F.Cu")
+		(net 4)
+	)
+	(segment
+		(start 182.48 121.52)
+		(end 182.88 121.92)
+		(width 0.2)
+		(layer "F.Cu")
+		(net 4)
+	)
+	(segment
+		(start 182.88 78.74)
+		(end 182.88 66.04)
+		(width 0.2)
+		(layer "F.Cu")
+		(net 4)
+	)
+	(segment
+		(start 175.26 99.06)
+		(end 172.68 99.06)
+		(width 0.2)
+		(layer "F.Cu")
+		(net 4)
+	)
+	(segment
+		(start 161.795 77.673683)
+		(end 167.64 71.828683)
+		(width 0.2)
+		(layer "F.Cu")
+		(net 4)
+	)
+	(segment
+		(start 149.82 55.88)
+		(end 152.4 55.88)
+		(width 0.2)
+		(layer "F.Cu")
+		(net 4)
+	)
+	(segment
+		(start 160.02 99.06)
+		(end 149.86 109.22)
+		(width 0.2)
+		(layer "F.Cu")
+		(net 4)
+	)
+	(segment
+		(start 175.26 48.26)
+		(end 180.34 53.34)
+		(width 0.2)
+		(layer "F.Cu")
+		(net 4)
+	)
+	(segment
+		(start 180.34 78.74)
+		(end 180.34 93.98)
+		(width 0.2)
+		(layer "F.Cu")
+		(net 4)
+	)
+	(segment
+		(start 157.48 139.7)
+		(end 162.56 139.7)
+		(width 0.2)
+		(layer "F.Cu")
+		(net 4)
+	)
+	(segment
+		(start 124.485 116.87)
+		(end 126.97 116.87)
+		(width 0.2)
+		(layer "F.Cu")
+		(net 4)
+	)
+	(segment
 		(start 159.98 116.84)
 		(end 167.64 116.84)
@@
 	)
 	(segment
-		(start 161.795 78.74)
-		(end 161.795 77.673683)
-		(width 0.2)
-		(layer "F.Cu")
-		(net 4)
-	)
-	(segment
-		(start 177.76 116.84)
-		(end 182.88 116.84)
-		(width 0.2)
-		(layer "F.Cu")
-		(net 4)
-	)
-	(segment
-		(start 182.88 111.76)
-		(end 175.26 104.14)
-		(width 0.2)
-		(layer "F.Cu")
-		(net 4)
-	)
-	(segment
-		(start 147.32 71.12)
-		(end 147.32 66.04)
-		(width 0.2)
-		(layer "F.Cu")
-		(net 4)
-	)
-	(segment
-		(start 172.72 139.7)
-		(end 172.72 137.16)
-		(width 0.2)
-		(layer "F.Cu")
-		(net 4)
-	)
-	(segment
-		(start 160.02 93.98)
-		(end 160.02 99.06)
-		(width 0.2)
-		(layer "F.Cu")
-		(net 4)
-	)
-	(segment
-		(start 137.16 71.12)
-		(end 147.32 71.12)
-		(width 0.2)
-		(layer "F.Cu")
-		(net 4)
-	)
-	(segment
-		(start 180.34 66.04)
-		(end 180.34 76.2)
-		(width 0.2)
-		(layer "F.Cu")
-		(net 4)
-	)
-	(segment
-		(start 180.34 76.2)
-		(end 177.8 78.74)
-		(width 0.2)
-		(layer "F.Cu")
-		(net 4)
-	)
-	(segment
-		(start 175.26 93.98)
-		(end 175.26 99.06)
-		(width 0.2)
-		(layer "F.Cu")
-		(net 4)
-	)
-	(segment
-		(start 177.8 78.74)
-		(end 180.34 78.74)
-		(width 0.2)
-		(layer "F.Cu")
-		(net 4)
-	)
-	(segment
-		(start 182.88 116.84)
-		(end 182.88 111.76)
-		(width 0.2)
-		(layer "F.Cu")
-		(net 4)
-	)
-	(segment
-		(start 137.16 124.46)
-		(end 167.64 124.46)
-		(width 0.2)
-		(layer "F.Cu")
-		(net 4)
-	)
-	(segment
-		(start 142.2 66.04)
-		(end 147.32 66.04)
-		(width 0.2)
-		(layer "F.Cu")
-		(net 4)
-	)
-	(segment
-		(start 152.4 55.88)
-		(end 152.4 66.04)
-		(width 0.2)
-		(layer "F.Cu")
-		(net 4)
-	)
-	(segment
-		(start 175.26 93.98)
-		(end 160.02 93.98)
-		(width 0.2)
-		(layer "F.Cu")
-		(net 4)
-	)
-	(segment
-		(start 167.64 124.46)
-		(end 167.64 139.7)
-		(width 0.2)
-		(layer "F.Cu")
-		(net 4)
-	)
-	(segment
-		(start 157.48 134.62)
-		(end 157.48 139.7)
-		(width 0.2)
-		(layer "F.Cu")
-		(net 4)
-	)
-	(segment
-		(start 182.88 66.04)
-		(end 180.3 66.04)
-		(width 0.2)
-		(layer "F.Cu")
-		(net 4)
-	)
-	(segment
-		(start 175.26 99.06)
-		(end 172.68 99.06)
-		(width 0.2)
-		(layer "F.Cu")
-		(net 4)
-	)
-	(segment
-		(start 161.795 77.673683)
-		(end 167.64 71.828683)
-		(width 0.2)
-		(layer "F.Cu")
-		(net 4)
-	)
-	(segment
-		(start 149.82 55.88)
-		(end 152.4 55.88)
-		(width 0.2)
-		(layer "F.Cu")
-		(net 4)
-	)
-	(segment
-		(start 160.02 99.06)
-		(end 149.86 109.22)
-		(width 0.2)
-		(layer "F.Cu")
-		(net 4)
-	)
-	(segment
-		(start 175.26 48.26)
-		(end 180.34 53.34)
-		(width 0.2)
-		(layer "F.Cu")
-		(net 4)
-	)
-	(segment
-		(start 180.34 78.74)
-		(end 180.34 93.98)
-		(width 0.2)
-		(layer "F.Cu")
-		(net 4)
-	)
-	(segment
-		(start 157.48 139.7)
-		(end 162.56 139.7)
-		(width 0.2)
-		(layer "F.Cu")
-		(net 4)
-	)
-	(segment
-		(start 124.485 116.87)
-		(end 126.97 116.87)
-		(width 0.2)
-		(layer "F.Cu")
-		(net 4)
-	)
-	(segment
 		(start 137.16 121.92)
 		(end 137.16 124.46)
@@
 	)
 	(segment
-		(start 177.8 119.38)
-		(end 177.8 116.88)
-		(width 0.2)
-		(layer "F.Cu")
-		(net 4)
-	)
-	(segment
 		(start 165.1 53.34)
 		(end 165.1 48.26)
@@
 	)
 	(segment
+		(start 167.64 121.52)
+		(end 182.48 121.52)
+		(width 0.2)
+		(layer "F.Cu")
+		(net 4)
+	)
+	(segment
 		(start 180.34 53.34)
 		(end 182.88 53.34)
@@
 		(width 0.2)
 		(layer "F.Cu")
-		(net 4)
-	)
-	(segment
-		(start 167.64 116.84)
-		(end 170.18 119.38)
-		(width 0.2)
-		(layer "F.Cu")
-		(net 4)
-	)
-	(segment
-		(start 170.18 119.38)
-		(end 177.8 119.38)
-		(width 0.2)
-		(layer "F.Cu")

Commit message: :sparkles: finish first pcb draft
Parts:
- added SW7: Joy_Button, Downloads:SW_BUTT-2, F.Cu at (177.3, 137.1)
- moved SW8 7.62 mm to (165.1, 134.7)
- moved SW6 6.30 mm to (156.3, 134.7)
- moved SW5 5.08 mm to (147.3, 134.6)
- moved SW13 3.51 mm to (155.9, 79.6)
- moved J3 2.49 mm to (144.7, 83.8)
- moved J4 2.49 mm to (129.4, 124.4)
- moved SW15 0.98 mm to (151.4, 99.1)
- moved SW16 0.69 mm to (175.2, 79.4)
- moved SW1 0.68 mm to (162.2, 66.6)
- moved SW2 0.66 mm to (177.3, 66.4)
- moved SW4 0.59 mm to (157.5, 117.4)
- moved SW3 0.58 mm to (175.2, 117.4)
Connections:
- J2 pad 3: /D7 -> /D5
- SW14 pad 1: /D0 -> /D5
- SW3 pad 1: /D1 -> /D4
- SW4 pad 1: /D17 -> /D3
Routing:
- net /GND: track 369.7 -> 413.3 mm
- net /D4: track 0.00 -> 39.5 mm
- net /D17: track 11.3 -> 43.3 mm
- net /D1: track 31.9 -> 0.00 mm
- net /D0: track 30.7 -> 0.00 mm
- net /D5: track 0.00 -> 29.1 mm
- net /D3: track 0.00 -> 19.3 mm
- net /D16: track 38.2 -> 25.2 mm
- net /D14: track 43.5 -> 34.9 mm
- net /D15: track 28.9 -> 21.1 mm
- net /VCC: track 57.0 -> 63.1 mm
- net /A1: track 23.5 -> 29.1 mm
- net /A2: track 27.1 -> 32.7 mm
- net /A0: track 27.5 -> 31.7 mm
- net /D8: track 51.4 -> 55.3 mm
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Other:
- outline, holes or cut-outs redrawn
- board text added: "susan <*)))><"
