File: pcb_designs/PCB Draft 1/4-7-2024.kicad_sch (KiCad schematic)
At the start: 19 parts, among them J1 Joystick_F_TH, J2 Joystick_B_TH, J3 Conn_01x17_Pin, J4 Conn_01x17_Pin, SW1 Left_Trigger, SW10 D_Pad_DOWN, SW11 D_Pad_LEFT, SW12 D_Pad_RIGHT, SW13 A_Button, SW14 X_Button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

Commit message: :sparkles: finish first pcb draft
Parts:
- added SW7: Joy_Button, Downloads:SW_BUTT-2, symbol Switch:SW_Push
Connections:
- net D0: no longer SW14.1
- net D1: no longer SW3.1
- net D17: now also SW7.1; no longer SW4.1
- net D3: now also SW4.1
- net D4: now also SW3.1
- net D5: now also J2.3 (Pin_3), SW14.1
- net D7: no longer J2.3 (Pin_3)
- net GND: now also SW7.2
Changed lines of the file:
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@@
+	(wire
+		(pts
+			(xy 201.93 55.88) (xy 205.74 55.88)
+		)
+		(stroke
+			(width 0)
+			(type default)
+		)
+	)
 	(wire
 		(pts
@@
 		(pts
 			(xy 166.37 119.38) (xy 156.21 119.38)
+		)
+		(stroke
+			(width 0)
+			(type default)
+		)
+	)
+	(wire
+		(pts
+			(xy 215.9 55.88) (xy 219.71 55.88)
 		)
 		(stroke
@@
 		)
 	)
+	(label "GND"
+		(at 215.9 55.88 0)
+		(fields_autoplaced yes)
+		(effects
+			(font
+				(size 1.27 1.27)
+			)
+			(justify left bottom)
+		)
+	)
 	(label "D1"
 		(at 143.51 111.76 0)
@@
 		)
 	)
-	(label "D7"
+	(label "D5"
 		(at 191.77 116.84 0)
 		(fields_autoplaced yes)
@@
 		)
 	)
-	(label "D17"
+	(label "D3"
 		(at 120.65 44.45 0)
 		(fields_autoplaced yes)
@@
 		)
 	)
-	(label "D0"
+	(label "D5"
 		(at 170.18 55.88 0)
 		(fields_autoplaced yes)
@@
 		)
 	)
+	(label "D17"
+		(at 201.93 55.88 0)
+		(fields_autoplaced yes)
+		(effects
+			(font
+				(size 1.27 1.27)
+			)
+			(justify left bottom)
+		)
+	)
 	(label "D16"
 		(at 142.24 116.84 0)
@@
 		)
 	)
-	(label "D1"
+	(label "D4"
 		(at 99.06 55.88 0)
 		(fields_autoplaced yes)
@@
 					(unit 1)
 				)
+			)
+		)
+	)
+	(symbol
+		(lib_id "Switch:SW_Push")
+		(at 210.82 55.88 0)
+		(unit 1)
+		(exclude_from_sim no)
+		(in_bom yes)
+		(on_board yes)
+		(dnp no)
+		(property "Reference" "SW7"
+			(at 210.82 48.26 0)
+			(effects
+				(font
+					(size 1.27 1.27)
+				)
+			)
+		)
+		(property "Value" "Joy_Button"
+			(at 210.82 50.8 0)
+			(effects
+				(font
+					(size 1.27 1.27)
+				)
+			)
+		)
+		(property "Footprint" "Downloads:SW_BUTT-2"
+			(at 210.82 50.8 0)
+			(effects
+				(font
+					(size 1.27 1.27)
+				)
+				(hide yes)
+			)
+		)
+		(property "Datasheet" "~"
+			(at 210.82 50.8 0)
+			(effects
+				(font
+					(size 1.27 1.27)
+				)
+				(hide yes)
+			)
+		)
+		(property "Description" "Push button switch, generic, two pins"
+			(at 210.82 55.88 0)
+			(effects
+				(font
+					(size 1.27 1.27)
+				)
+				(hide yes)
+			)
+		)
+		(pin "2"
+		)
+		(pin "1"
+		)
+		(instances
+			(project "3-24-2024"
+				(path "/dac850b7-79d7-4b35-b972-5350d8cb3bcd"
+					(reference "SW7")
+					(unit 1)
+				)
