File: 2024_fall/PCB Order 3/Front PCB/ohgc_front_pcb.kicad_pcb (KiCad board)
At the start: 2 copper layers, 67 x 88.9 mm, 11 parts, among them J1 d-pad pins, J2 misc pins, J3 joytick pins, J4 joystick, SW1 Up, SW2 Down, SW3 Left, SW4 Right, SW6 Home, SW7 Start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

Commit message: :construction: remove joystick from front pcb
Parts:
- removed J3: joytick pins, Connector_PinSocket_2.54mm:PinSocket_1x05_P2.54mm_Vertical
- removed J4: joystick, Connector_PinSocket_2.54mm:PinSocket_1x05_P2.54mm_Vertical
Routing:
- net /A2: track 73.1 -> 0.00 mm
- net /VCC: track 67.8 -> 0.00 mm
- net /GND: track 183.6 -> 117.5 mm
- net /A1: track 62.3 -> 0.00 mm
- net /A0: track 52.4 -> 0.00 mm
Other:
- board size 67 x 88.9 mm -> 67 x 59.3 mm
