File: 2026_spring/pcb/back_pcb.kicad_sch (KiCad schematic)
At the start: 20 parts, among them J1 front joystick, J2 bottom joystick, J3 Arduino, J4 Arduino, SW1 Left Trigger, SW10 Home, SW11 Start, SW13 A, SW14 X, SW15 Y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

Commit message: :construction: fix screw terminals
Parts:
- J2: footprint Connector_PinSocket_2.54mm:PinSocket_1x05_P2.54mm_Vertical_SMD_Pin1Left -> Downloads:TE_282837-5; symbol Connector:Conn_01x05_Socket -> Connector:Screw_Terminal_01x05
Connections:
- net A3: now also J2.2 (Pin_2); no longer J1.B1A (SEL+), J2.3 (Pin_3)
- net A5: now also J2.3 (Pin_3); no longer J2.2 (Pin_2)
- net D7: now also J1.B1A (SEL+)
Changed lines of the file:
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@@
 		)
 	)
-	(label "A3"
+	(label "A5"
 		(at 191.77 116.84 0)
 		(fields_autoplaced yes)
@@
 		)
 	)
-	(label "A5"
+	(label "A3"
 		(at 191.77 114.3 0)
 		(fields_autoplaced yes)
@@
 		)
 	)
-	(label "A3"
+	(label "D7"
 		(at 148.59 156.21 0)
 		(fields_autoplaced yes)
@@
 	)
 	(symbol
-		(lib_id "Connector:Conn_01x05_Socket")
+		(lib_id "Connector:Screw_Terminal_01x05")
 		(at 203.2 116.84 0)
 		(unit 1)
@@
 		(fields_autoplaced yes)
 		(property "Reference" "J2"
-			(at 204.47 115.5699 0)
+			(at 205.74 115.5699 0)
 			(effects
 				(font
@@
 		)
 		(property "Value" "bottom joystick"
-			(at 204.47 118.1099 0)
+			(at 205.74 118.1099 0)
 			(effects
 				(font
@@
 			)
 		)
-		(property "Footprint" "Connector_PinSocket_2.54mm:PinSocket_1x05_P2.54mm_Vertical_SMD_Pin1Left"
+		(property "Footprint" "Downloads:TE_282837-5"
 			(at 203.2 116.84 0)
 			(effects
@@
 			)
 		)
-		(property "Description" ""
+		(property "Description" "Generic screw terminal, single row, 01x05, script generated (kicad-library-utils/schlib/autogen/connector/)"
 			(at 203.2 116.84 0)
 			(effects

Commit message: :sparkle: move arduino to middle of pcb
Parts:
- added D1: LED, Downloads:LEDRD254W57D500H1070, symbol Device:LED
- added R1: R_Small, Resistor_THT:R_Axial_DIN0204_L3.6mm_D1.6mm_P1.90mm_Vertical, symbol Device:R_Small
- SW1, SW10, SW11, SW13, SW14, SW15, SW16, SW17, SW2, SW3, SW4, SW5, SW6, SW7, SW8, SW9: footprint Button_Switch_SMD:SW_DIP_SPSTx01_Slide_Copal_CHS-01A_W5.08mm_P1.27mm_JPin -> Downloads:SW_PTS636_SM43J_SMTR_LFS
Connections:
- net D2: now also R1.2
- net GND: now also D1.1 (K)
- new net R1: D1.2 (A), R1.1
Changed lines of the file:
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@@
 	(wire
 		(pts
+			(xy 191.77 27.94) (xy 194.31 27.94)
+		)
+		(stroke
+			(width 0)
+			(type default)
+		)
+	)
+	(wire
+		(pts
 			(xy 196.85 44.45) (xy 200.66 44.45)
 		)
@@
 	(wire
 		(pts
+			(xy 185.42 27.94) (xy 187.96 27.94)
+		)
+		(stroke
+			(width 0)
+			(type default)
+		)
+	)
+	(wire
+		(pts
 			(xy 116.84 111.76) (xy 123.19 111.76)
 		)
@@
 	(wire
 		(pts
+			(xy 199.39 27.94) (xy 203.2 27.94)
+		)
+		(stroke
+			(width 0)
+			(type default)
+		)
+	)
+	(wire
+		(pts
 			(xy 123.19 91.44) (xy 116.84 91.44)
 		)
@@
 		)
 	)
+	(label "R1"
+		(at 191.77 27.94 0)
+		(fields_autoplaced yes)
+		(effects
+			(font
+				(size 1.27 1.27)
+			)
+			(justify left bottom)
+		)
+	)
 	(label "VCC"
 		(at 119.38 104.14 180)
@@
 		)
 	)
+	(label "GND"
+		(at 177.8 27.94 0)
+		(fields_autoplaced yes)
+		(effects
+			(font
+				(size 1.27 1.27)
+			)
+			(justify left bottom)
+		)
+	)
 	(label "D3"
 		(at 143.51 99.06 0)
@@
 		)
 	)
+	(label "R1"
+		(at 187.96 27.94 0)
+		(fields_autoplaced yes)
+		(effects
+			(font
+				(size 1.27 1.27)
+			)
+			(justify left bottom)
+		)
+	)
 	(label "GND"
 		(at 236.22 50.8 0)
@@
 		)
 	)
+	(label "D2"
+		(at 203.2 27.94 0)
+		(fields_autoplaced yes)
+		(effects
+			(font
+				(size 1.27 1.27)
+			)
+			(justify left bottom)
+		)
+	)
 	(label "GND"
 		(at 196.85 44.45 0)
@@
 			)
 		)
-		(property "Footprint" "Button_Switch_SMD:SW_DIP_SPSTx01_Slide_Copal_CHS-01A_W5.08mm_P1.27mm_JPin"
+		(property "Footprint" "Downloads:SW_PTS636_SM43J_SMTR_LFS"
 			(at 251.46 45.72 0)
 			(effects
@@
 			)
 		)
-		(property "Footprint" "Button_Switch_SMD:SW_DIP_SPSTx01_Slide_Copal_CHS-01A_W5.08mm_P1.27mm_JPin"
+		(property "Footprint" "Downloads:SW_PTS636_SM43J_SMTR_LFS"
 			(at 171.45 39.37 0)
 			(effects
@@
 			)
 		)
-		(property "Footprint" "Button_Switch_SMD:SW_DIP_SPSTx01_Slide_Copal_CHS-01A_W5.08mm_P1.27mm_JPin"
+		(property "Footprint" "Downloads:SW_PTS636_SM43J_SMTR_LFS"
 			(at 231.14 45.72 0)
 			(effects
@@
 			)
 		)
-		(property "Footprint" "Button_Switch_SMD:SW_DIP_SPSTx01_Slide_Copal_CHS-01A_W5.08mm_P1.27mm_JPin"
+		(property "Footprint" "Downloads:SW_PTS636_SM43J_SMTR_LFS"
 			(at 87.63 39.37 0)
 			(effects
@@
 			)
 		)
-		(property "Footprint" "Button_Switch_SMD:SW_DIP_SPSTx01_Slide_Copal_CHS-01A_W5.08mm_P1.27mm_JPin"
+		(property "Footprint" "Downloads:SW_PTS636_SM43J_SMTR_LFS"
 			(at 213.36 39.37 0)
 			(effects
@@
 			)
 		)
-		(property "Footprint" "Button_Switch_SMD:SW_DIP_SPSTx01_Slide_Copal_CHS-01A_W5.08mm_P1.27mm_JPin"
+		(property "Footprint" "Downloads:SW_PTS636_SM43J_SMTR_LFS"
 			(at 107.95 50.8 0)
 			(effects
@@
 			)
 		)
-		(property "Footprint" "Button_Switch_SMD:SW_DIP_SPSTx01_Slide_Copal_CHS-01A_W5.08mm_P1.27mm_JPin"
+		(property "Footprint" "Downloads:SW_PTS636_SM43J_SMTR_LFS"
 			(at 168.91 74.93 0)
 			(effects
@@
 	)
 	(symbol
+		(lib_id "Device:LED")
+		(at 181.61 27.94 0)
+		(unit 1)
+		(exclude_from_sim no)
+		(in_bom yes)
+		(on_board yes)
+		(dnp no)
+		(fields_autoplaced yes)
+		(property "Reference" "D1"
+			(at 180.0225 21.59 0)
+			(effects
+				(font
+					(size 1.27 1.27)
+				)
+			)
+		)
+		(property "Value" "LED"
+			(at 180.0225 24.13 0)
+			(effects
+				(font
+					(size 1.27 1.27)
+				)
+			)
+		)
+		(property "Footprint" "Downloads:LEDRD254W57D500H1070"
+			(at 181.61 27.94 0)
+			(effects
+				(font
+					(size 1.27 1.27)
+				)
+				(hide yes)
+			)
+		)
+		(property "Datasheet" "~"
+			(at 181.61 27.94 0)
+			(effects
+				(font
+					(size 1.27 1.27)
+				)
+				(hide yes)
+			)
+		)
+		(property "Description" "Light emitting diode"
+			(at 181.61 27.94 0)
+			(effects
+				(font
+					(size 1.27 1.27)
+				)
+				(hide yes)
+			)
+		)
+		(pin "2"
+		)
+		(pin "1"
+		)
+		(instances
+			(project "back_pcb"
+				(path "/dac850b7-79d7-4b35-b972-5350d8cb3bcd"
+					(reference "D1")
+					(unit 1)
+				)
+			)
+		)
+	)
+	(symbol
 		(lib_id "Switch:SW_Push")
 		(at 107.95 44.45 0)
@@
 			)
 		)
-		(property "Footprint" "Button_Switch_SMD:SW_DIP_SPSTx01_Slide_Copal_CHS-01A_W5.08mm_P1.27mm_JPin"
+		(property "Footprint" "Downloads:SW_PTS636_SM43J_SMTR_LFS"
 			(at 107.95 39.37 0)
 			(effects
@@
 			)
 		)
-		(property "Footprint" "Button_Switch_SMD:SW_DIP_SPSTx01_Slide_Copal_CHS-01A_W5.08mm_P1.27mm_JPin"
+		(property "Footprint" "Downloads:SW_PTS636_SM43J_SMTR_LFS"
 			(at 129.54 39.37 0)
 			(effects
@@
 			)
 		)
-		(property "Footprint" "Button_Switch_SMD:SW_DIP_SPSTx01_Slide_Copal_CHS-01A_W5.08mm_P1.27mm_JPin"
+		(property "Footprint" "Downloads:SW_PTS636_SM43J_SMTR_LFS"
 			(at 273.05 45.72 0)
 			(effects
@@
 			)
 		)
-		(property "Footprint" "Button_Switch_SMD:SW_DIP_SPSTx01_Slide_Copal_CHS-01A_W5.08mm_P1.27mm_JPin"
+		(property "Footprint" "Downloads:SW_PTS636_SM43J_SMTR_LFS"
 			(at 191.77 39.37 0)
 			(effects
@@
 	)
 	(symbol
+		(lib_id "Device:R_Small")
+		(at 196.85 27.94 90)
+		(unit 1)
+		(exclude_from_sim no)
+		(in_bom yes)
+		(on_board yes)
+		(dnp no)
+		(fields_autoplaced yes)
+		(property "Reference" "R1"
+			(at 196.85 22.86 90)
+			(effects
+				(font
+					(size 1.27 1.27)
+				)
+			)
+		)
+		(property "Value" "R_Small"
+			(at 196.85 25.4 90)
+			(effects
+				(font
+					(size 1.27 1.27)
+				)
+			)
+		)
+		(property "Footprint" "Resistor_THT:R_Axial_DIN0204_L3.6mm_D1.6mm_P1.90mm_Vertical"
+			(at 196.85 27.94 0)
+			(effects
+				(font
+					(size 1.27 1.27)
+				)
+				(hide yes)
+			)
+		)
+		(property "Datasheet" "~"
+			(at 196.85 27.94 0)
+			(effects
+				(font
+					(size 1.27 1.27)
+				)
+				(hide yes)
+			)
+		)
+		(property "Description" "Resistor, small symbol"
+			(at 196.85 27.94 0)
+			(effects
+				(font
+					(size 1.27 1.27)
+				)
+				(hide yes)
+			)
+		)
+		(pin "2"
+		)
+		(pin "1"
+		)
+		(instances
+			(project "back_pcb"
+				(path "/dac850b7-79d7-4b35-b972-5350d8cb3bcd"
+					(reference "R1")
+					(unit 1)
+				)
+			)
+		)
+	)
+	(symbol
 		(lib_id "Switch:SW_Push")
 		(at 191.77 55.88 0)
@@
 			)
 		)
-		(property "Footprint" "Button_Switch_SMD:SW_DIP_SPSTx01_Slide_Copal_CHS-01A_W5.08mm_P1.27mm_JPin"
+		(property "Footprint" "Downloads:SW_PTS636_SM43J_SMTR_LFS"
 			(at 191.77 50.8 0)
 			(effects
@@
 			)
 		)
-		(property "Footprint" "Button_Switch_SMD:SW_DIP_SPSTx01_Slide_Copal_CHS-01A_W5.08mm_P1.27mm_JPin"
+		(property "Footprint" "Downloads:SW_PTS636_SM43J_SMTR_LFS"
 			(at 189.23 74.93 0)
 			(effects
@@
 			)
 		)
-		(property "Footprint" "Button_Switch_SMD:SW_DIP_SPSTx01_Slide_Copal_CHS-01A_W5.08mm_P1.27mm_JPin"
+		(property "Footprint" "Downloads:SW_PTS636_SM43J_SMTR_LFS"
 			(at 203.2 90.17 0)
 			(effects
@@
 			)
 		)
-		(property "Footprint" "Button_Switch_SMD:SW_DIP_SPSTx01_Slide_Copal_CHS-01A_W5.08mm_P1.27mm_JPin"
+		(property "Footprint" "Downloads:SW_PTS636_SM43J_SMTR_LFS"
 			(at 210.82 74.93 0)
 			(effects
@@
 			)
 		)
-		(property "Footprint" "Button_Switch_SMD:SW_DIP_SPSTx01_Slide_Copal_CHS-01A_W5.08mm_P1.27mm_JPin"
+		(property "Footprint" "Downloads:SW_PTS636_SM43J_SMTR_LFS"
 			(at 171.45 90.17 0)
 			(effects
